Commit message: Add files via upload

File: description/profile_channel.xacro (robot description, xacro)
@@ -1,4 +1,4 @@
 <?xml version="1.0"?>
-<robot xmlns:xacro="http://www.ros.org/wiki/xacro"  name="robot">
+<robot xmlns:xacro="http://www.ros.org/wiki/xacro">
     <xacro:include filename="inertial_macros.xacro"/>
     <xacro:macro name="profile_channel" params="parent child profile_mass profile_length profile_width profile_height xyz rpy">

File: description/robot_core.xacro (robot description, xacro)
@@ -2,5 +2,8 @@
 <robot xmlns:xacro="http://www.ros.org/wiki/xacro" >
     <xacro:include filename="profile_channel.xacro"/>
-    <link name="base_link"></link>
+    <xacro:include filename="wheel.xacro"/>
+    <link name="base_link">
+    </link>
+    <!-- Chassis profile Channels -->
     <xacro:property name="Chassis_profile_size" value="0.02"/>
     <xacro:property name="Chassis_profile_length" value="0.560"/>
@@ -27,3 +30,8 @@
     <xacro:profile_channel parent="base_link" child="left_top_motor_support_profile_channel"     profile_mass="0.002" profile_length="${motor_support_profile_length}" profile_width="${Chassis_profile_size}"  profile_height="${Chassis_profile_size}"  xyz=" 0.0475 -0.205   0.070"  rpy="0 0 0"/>
     <xacro:profile_channel parent="base_link" child="right_top_motor_support_profile_channel"    profile_mass="0.002" profile_length="${motor_support_profile_length}" profile_width="${Chassis_profile_size}"  profile_height="${Chassis_profile_size}"  xyz="-0.0475  0.205   0.070"  rpy="0 0 0"/>
+    <!-- Omni Wheels-->
+    <xacro:omni_wheel parent="base_link" child="front"  xyz=" 0.255   0.205 0.035"  rpy=" 0.0   1.57 0.0 "/>
+    <xacro:omni_wheel parent="base_link" child="back"   xyz="-0.255  -0.205 0.035"  rpy=" 0.0  -1.57 0.0"/>
+    <xacro:omni_wheel parent="base_link" child="left"   xyz="-0.205  0.255 0.035"   rpy="-1.57  0    0.0"/>
+    <xacro:omni_wheel parent="base_link" child="right"  xyz=" 0.205 -0.255 0.035"   rpy=" 1.57  0    0.0"/>
 </robot>

Commit message: Update profile_channel.xacro

File: description/profile_channel.xacro (robot description, xacro)
@@ -19,5 +19,5 @@
             </collision>
             <xacro:inertial_box mass="${profile_mass}" x="${profile_length}" y="${profile_width}" z="${profile_height}">
-                <origin xyz="${profile_length/2} 0 ${profile_height/2}" rpy="${rpy}"/>
+                <origin xyz="0 0 0" rpy="0 0 0"/>
             </xacro:inertial_box>
         </link>
