Commit message: Update wheel.xacro

File: description/wheel.xacro (robot description, xacro)
@@ -10,5 +10,5 @@
                 <origin xyz="0.0 0.0 0.0" rpy="0.0 0.0 0.0"/>
                 <geometry>
-                    <cylinder radius="${wheel_radius}" length="${wheel_thickness}"/>
+                    <mesh filename="file://$(find project_eva)/meshes/wheel_roller.STL"/>
                 </geometry>
                 <material name="black">

Commit message: Update wheel.xacro

File: description/wheel.xacro (robot description, xacro)
@@ -10,5 +10,6 @@
                 <origin xyz="0.0 0.0 0.0" rpy="0.0 0.0 0.0"/>
                 <geometry>
-                    <mesh filename="file://$(find project_eva)/meshes/wheel_roller.STL"/>
+                    <cylinder radius="${wheel_radius}" length="${wheel_thickness}"/>
+                    <!--<mesh filename="file://$(find project_eva)/meshes/omni_wheel.STL"/>-->
                 </geometry>
                 <material name="black">

Commit message: Update wheel.xacro

File: description/wheel.xacro (robot description, xacro)
@@ -1,4 +1,4 @@
 <?xml version="1.0"?>
-<robot xmlns:xacro="http://www.ros.org/wiki/xacro"  name="robot">
+<robot xmlns:xacro="http://www.ros.org/wiki/xacro">
     <xacro:include filename="inertial_macros.xacro"/>
     <xacro:property name="wheel_mass" value="0.650"/>
@@ -11,5 +11,5 @@
                 <geometry>
                     <cylinder radius="${wheel_radius}" length="${wheel_thickness}"/>
-                    <!--<mesh filename="file://$(find project_eva)/meshes/omni_wheel.STL"/>-->
+                    <!-- <mesh filename="file://$(find project_eva)/meshes/omni_wheel.STL"/> -->
                 </geometry>
                 <material name="black">
@@ -28,6 +28,8 @@
             </xacro:inertial_cylinder>
         </link>
-        <gazebo reference = "wheel_${child}_link">
+        <gazebo reference = "${child}_wheel_link">
             <material>Gazebo/Black</material>
+            <!-- <mu1 value="0.001"/>
+            <mu2 value="0.001"/> -->
         </gazebo>
         <joint name="${child}_wheel_joint" type="continuous">

Commit message: Update wheel.xacro

File: description/wheel.xacro (robot description, xacro)
@@ -7,5 +7,5 @@
     <xacro:macro name="wheel" params="parent child xyz rpy">
         <link name="${child}_wheel_link">
-            <visual name="">
+            <visual>
                 <origin xyz="0.0 0.0 0.0" rpy="0.0 0.0 0.0"/>
                 <geometry>
@@ -30,6 +30,6 @@
         <gazebo reference = "${child}_wheel_link">
             <material>Gazebo/Black</material>
-            <!-- <mu1 value="0.001"/>
-            <mu2 value="0.001"/> -->
+            <mu1 value="0.001"/>
+            <mu2 value="0.001"/>
         </gazebo>
         <joint name="${child}_wheel_joint" type="continuous">
