Commit message: Add files via upload

File: description/omni_wheel.xacro (robot description, xacro)
@@ -16,14 +16,10 @@
                 <origin xyz="0 0 0" rpy="1.57 0 0" />
                 <geometry>
-                    <mesh filename="file://$(find project_eva)/meshes/wheel_roller.STL"/>
+                    <sphere radius="0.0095"/>
                 </geometry>
             </collision>
-            <inertial>
-                <origin xyz="5.09395238803556E-16 6.79977710486667E-16 -0.0104983350650447" rpy="1.57 0 0" />
-                <mass value="0.002" />
-                <inertia ixx="0.000781592793267822" ixy="1.05247463532391E-18" ixz="-6.56787240457889E-19"
-                         iyy="0.000781592793267821" iyz="-1.19446449980815E-19"
-                         izz="0.0014442649663699" />
-            </inertial>
+            <xacro:inertial_cylinder mass="0.005" length="0.018" radius="0.0095">
+                <origin xyz="0 0 0" rpy="0 0 0"/>
+            </xacro:inertial_cylinder>
         </link>
         <joint name="${parent}_${child}_joint" type="continuous">
@@ -56,6 +52,6 @@
             </collision>
             <inertial>
-                <origin xyz="5.09395238803556E-16 6.79977710486667E-16 -0.0104983350650447" rpy="${rpy}" />
-                <mass value="0.25" />
+                <origin xyz="0 0 -0.0045" rpy="${rpy}" />
+                <mass value="0.1625" />
                 <inertia ixx="0.000781592793267822" ixy="7.25426890587709E-19" ixz="-6.09681598211934E-19"
                         iyy="0.000781592793267821" iyz="-1.67393264409733E-19"

File: description/robot.urdf.xacro (robot description, xacro)
@@ -1,4 +1,5 @@
 <?xml version="1.0"?>
 <robot xmlns:xacro="http://www.ros.org/wiki/xacro"  name="robot">
+    <xacro:arg name="use_omni_wheel" default="false"/>
     <xacro:include filename="robot_core.xacro"/>
     <!-- <xacro:include filename="gazebo_control.xacro"/> -->

File: description/robot_core.xacro (robot description, xacro)
@@ -2,6 +2,4 @@
 <robot xmlns:xacro="http://www.ros.org/wiki/xacro" >
     <xacro:include filename="profile_channel.xacro"/>
-    <xacro:include filename="omni_wheel.xacro"/>
-    <xacro:include filename="wheel.xacro"/>
     <!-- Base Link -->
     <link name="base_link">
@@ -34,13 +32,20 @@
     <!-- Bot Front Marker -->
     <xacro:profile_channel parent="base_link" child="Bot_Front_Marker_profile_channel"   profile_mass="0.001" profile_length="${Chassis_side_profile_length}" profile_width="${Chassis_profile_size}"  profile_height="${Chassis_profile_size}"  xyz="0.290  0  0.105"  rpy="0 -1.57 0"/>
-    <!-- Omni Wheels-->
-    <xacro:omni_wheel parent="base_link" child="front_left"  xyz=" 0.255   0.205 0.035"  rpy=" 0.0   1.57 0.0 "/>
-    <xacro:omni_wheel parent="base_link" child="back_right"   xyz="-0.255  -0.205 0.035"  rpy=" 0.0  -1.57 0.0"/>
-    <xacro:omni_wheel parent="base_link" child="back_left"   xyz="-0.205  0.255 0.035"   rpy="-1.57  0    0.0"/>
-    <xacro:omni_wheel parent="base_link" child="front_right"  xyz=" 0.205 -0.255 0.035"   rpy=" 1.57  0    0.0"/>
     <!-- Wheels-->
-    <!--<xacro:wheel parent="base_link" child="front_left"  xyz=" 0.245   0.205 0.035"  rpy=" 0.0   1.57 0.0 "/>
-    <xacro:wheel parent="base_link" child="back_right"   xyz="-0.245  -0.205 0.035"  rpy=" 0.0  -1.57 0.0"/>
-    <xacro:wheel parent="base_link" child="back_left"   xyz="-0.205  0.245 0.035"   rpy="-1.57  0    0.0"/>
-    <xacro:wheel parent="base_link" child="front_right"  xyz=" 0.205 -0.245 0.035"   rpy=" 1.57  0    0.0"/>-->
+    <xacro:if value="$(arg use_omni_wheel)">
+        <!-- Omni Wheels -->
+        <xacro:include filename="omni_wheel.xacro"/>
+        <xacro:omni_wheel parent="base_link" child="front_left"  xyz=" 0.255   0.205 0.035"  rpy=" 0.0   1.57 0.0 "/>
+        <xacro:omni_wheel parent="base_link" child="back_right"   xyz="-0.255  -0.205 0.035"  rpy=" 0.0  -1.57 0.0"/>
+        <xacro:omni_wheel parent="base_link" child="back_left"   xyz="-0.205  0.255 0.035"   rpy="-1.57  0    0.0"/>
+        <xacro:omni_wheel parent="base_link" child="front_right"  xyz=" 0.205 -0.255 0.035"   rpy=" 1.57  0    0.0"/>
+    </xacro:if>
+    <xacro:unless value="$(arg use_omni_wheel)">
+        <!--Normal Wheels-->
+        <xacro:include filename="wheel.xacro"/>
+        <xacro:wheel parent="base_link" child="front_left"  xyz=" 0.245   0.205 0.035"  rpy=" 0.0   1.57 0.0 "/>
+        <xacro:wheel parent="base_link" child="back_right"   xyz="-0.245  -0.205 0.035"  rpy=" 0.0  -1.57 0.0"/>
+        <xacro:wheel parent="base_link" child="back_left"   xyz="-0.205  0.245 0.035"   rpy="-1.57  0    0.0"/>
+        <xacro:wheel parent="base_link" child="front_right"  xyz=" 0.205 -0.245 0.035"   rpy=" 1.57  0    0.0"/>
+    </xacro:unless>
 </robot>

Commit message: Add files via upload

File: description/omni_wheel.xacro (robot description, xacro)
@@ -7,5 +7,5 @@
                 <origin xyz="0 0 0" rpy="1.57 0 0" />
                 <geometry>
-                    <mesh filename="file://$(find project_eva)/meshes/wheel_roller.STL"/>
+                    <mesh filename="file://$(find project_eva)/meshes/Drive/wheel_roller.STL"/>
                 </geometry>
                 <material name="wheel_rubber">
@@ -16,14 +16,10 @@
                 <origin xyz="0 0 0" rpy="1.57 0 0" />
                 <geometry>
-                    <mesh filename="file://$(find project_eva)/meshes/wheel_roller.STL"/>
+                    <sphere radius="0.0095"/>
                 </geometry>
             </collision>
-            <inertial>
-                <origin xyz="5.09395238803556E-16 6.79977710486667E-16 -0.0104983350650447" rpy="1.57 0 0" />
-                <mass value="0.002" />
-                <inertia ixx="0.000781592793267822" ixy="1.05247463532391E-18" ixz="-6.56787240457889E-19"
-                         iyy="0.000781592793267821" iyz="-1.19446449980815E-19"
-                         izz="0.0014442649663699" />
-            </inertial>
+            <xacro:inertial_cylinder mass="0.005" length="0.018" radius="0.0095">
+                <origin xyz="0 0 0" rpy="0 0 0"/>
+            </xacro:inertial_cylinder>
         </link>
         <joint name="${parent}_${child}_joint" type="continuous">
@@ -43,5 +39,5 @@
                 <origin xyz="${xyz}" rpy="${rpy}"/>
                 <geometry>
-                    <mesh filename="file://$(find project_eva)/meshes/wheel_link.STL"/>
+                    <mesh filename="file://$(find project_eva)/meshes/Drive/wheel_link.STL"/>
                 </geometry>
                 <material name="">
@@ -52,10 +48,10 @@
                 <origin xyz="${xyz}" rpy="${rpy}"/>
                 <geometry>
-                    <mesh filename="file://$(find project_eva)/meshes/wheel_link.STL"/>
+                    <mesh filename="file://$(find project_eva)/meshes/Drive/wheel_link.STL"/>
                 </geometry>
             </collision>
             <inertial>
-                <origin xyz="5.09395238803556E-16 6.79977710486667E-16 -0.0104983350650447" rpy="${rpy}" />
-                <mass value="0.25" />
+                <origin xyz="0 0 -0.0045" rpy="${rpy}" />
+                <mass value="0.1625" />
                 <inertia ixx="0.000781592793267822" ixy="7.25426890587709E-19" ixz="-6.09681598211934E-19"
                         iyy="0.000781592793267821" iyz="-1.67393264409733E-19"

File: description/robot.urdf.xacro (robot description, xacro)
@@ -1,5 +1,10 @@
 <?xml version="1.0"?>
 <robot xmlns:xacro="http://www.ros.org/wiki/xacro"  name="robot">
+    <xacro:arg name="use_omni_wheel" default="false"/>
     <xacro:include filename="robot_core.xacro"/>
+    <xacro:include filename="arm.xacro"/>
+    <xacro:include filename="body.xacro"/>
+    <xacro:include filename="leg.xacro"/>
+    <xacro:include filename="realsense.xacro"/>
     <!-- <xacro:include filename="gazebo_control.xacro"/> -->
     <!-- <xacro:include filename="ros2_control.xacro"/> -->

File: description/robot_core.xacro (robot description, xacro)
@@ -2,13 +2,18 @@
 <robot xmlns:xacro="http://www.ros.org/wiki/xacro" >
     <xacro:include filename="profile_channel.xacro"/>
-    <xacro:include filename="omni_wheel.xacro"/>
-    <xacro:include filename="wheel.xacro"/>
     <!-- Base Link -->
     <link name="base_link">
     </link>
+    <link name="EVA_base_link">
+    </link>
+    <joint name="base_joint" type="fixed">
+        <parent link="base_link"/>
+        <child link="EVA_base_link"/>
+        <origin xyz="0 0 0.140" rpy="0 0 0" />
+    </joint>
     <!-- Chassis profile Channels -->
     <xacro:property name="Chassis_profile_size" value="0.02"/>
     <xacro:property name="Chassis_profile_length" value="0.560"/>
-    <xacro:property name="Chassis_side_profile_length" value="0.090"/>
+    <xacro:property name="Chassis_side_profile_length" value="0.150"/>
     <xacro:property name="motor_support_profile_length" value="0.485"/>
     <xacro:profile_channel parent="base_link" child="front_bottom_profile_channel" profile_mass="0.28" profile_length="${Chassis_profile_length}" profile_width="${Chassis_profile_size}"  profile_height="${Chassis_profile_size}"  xyz=" 0.290   0.00  0.00"   rpy="0 0 -1.57" />
@@ -18,29 +23,36 @@
     <xacro:profile_channel parent="base_link" child="front_bottom_motor_support_profile_channel" profile_mass="0.2425" profile_length="${motor_support_profile_length}" profile_width="${Chassis_profile_size}"  profile_height="${Chassis_profile_size}"  xyz=" 0.205   0.0475  0.00"   rpy="0 0 -1.57"/>
     <xacro:profile_channel parent="base_link" child="back_bottom_motor_support_profile_channel"  profile_mass="0.2425" profile_length="${motor_support_profile_length}" profile_width="${Chassis_profile_size}"  profile_height="${Chassis_profile_size}"  xyz="-0.205  -0.0475  0.00"   rpy="0 0 -1.57"/>
-    <xacro:profile_channel parent="base_link" child="left_bottom_motor_support_profile_channel"  profile_mass="0.2425" profile_length="${motor_support_profile_length}" profile_width="${Chassis_profile_size}"  profile_height="${Chassis_profile_size}"  xyz=" 0.0475 -0.205   0.00"   rpy="0 0 0" />
-    <xacro:profile_channel parent="base_link" child="right_bottom_motor_support_profile_channel" profile_mass="0.2425" profile_length="${motor_support_profile_length}" profile_width="${Chassis_profile_size}"  profile_height="${Chassis_profile_size}"  xyz="-0.0475  0.205   0.00"   rpy="0 0 0" />
-    <xacro:profile_channel parent="base_link" child="front_top_profile_channel" profile_mass="0.28" profile_length="${Chassis_profile_length}" profile_width="${Chassis_profile_size}"  profile_height="${Chassis_profile_size}"  xyz=" 0.290   0.00  0.070"   rpy="0 0 -1.57" />
-    <xacro:profile_channel parent="base_link" child="back_top_profile_channel"  profile_mass="0.28" profile_length="${Chassis_profile_length}" profile_width="${Chassis_profile_size}"  profile_height="${Chassis_profile_size}"  xyz="-0.290   0.00  0.070"    rpy="0 0 -1.57" />
-    <xacro:profile_channel parent="base_link" child="left_top_profile_channel"  profile_mass="0.28" profile_length="${Chassis_profile_length}" profile_width="${Chassis_profile_size}"  profile_height="${Chassis_profile_size}"  xyz=" 0.0     0.290 0.070"  rpy="0 0 0" />
-    <xacro:profile_channel parent="base_link" child="right_top_profile_channel" profile_mass="0.28" profile_length="${Chassis_profile_length}" profile_width="${Chassis_profile_size}"  profile_height="${Chassis_profile_size}"  xyz=" 0.0    -0.290 0.070"  rpy="0 0 0" />
-    <xacro:profile_channel parent="base_link" child="front_top_motor_support_profile_channel"    profile_mass="0.2425" profile_length="${motor_support_profile_length}" profile_width="${Chassis_profile_size}"  profile_height="${Chassis_profile_size}"  xyz=" 0.205   0.0475  0.070"  rpy="0 0 -1.57"/>
-    <xacro:profile_channel parent="base_link" child="back_top_motor_support_profile_channel"     profile_mass="0.2425" profile_length="${motor_support_profile_length}" profile_width="${Chassis_profile_size}"  profile_height="${Chassis_profile_size}"  xyz="-0.205  -0.0475  0.070"  rpy="0 0 -1.57"/>
-    <xacro:profile_channel parent="base_link" child="left_top_motor_support_profile_channel"     profile_mass="0.2425" profile_length="${motor_support_profile_length}" profile_width="${Chassis_profile_size}"  profile_height="${Chassis_profile_size}"  xyz=" 0.0475 -0.205   0.070"  rpy="0 0 0"/>
-    <xacro:profile_channel parent="base_link" child="right_top_motor_support_profile_channel"    profile_mass="0.2425" profile_length="${motor_support_profile_length}" profile_width="${Chassis_profile_size}"  profile_height="${Chassis_profile_size}"  xyz="-0.0475  0.205   0.070"  rpy="0 0 0"/>
-    <xacro:profile_channel parent="base_link" child="front_left_side_support_profile_channel"   profile_mass="0.045" profile_length="${Chassis_side_profile_length}" profile_width="${Chassis_profile_size}"  profile_height="${Chassis_profile_size}"  xyz=" 0.290   0.290  0.035" rpy="0 -1.57 0"/>
-    <xacro:profile_channel parent="base_link" child="front_right_side_support_profile_channel"  profile_mass="0.045" profile_length="${Chassis_side_profile_length}" profile_width="${Chassis_profile_size}"  profile_height="${Chassis_profile_size}"  xyz=" 0.290  -0.290  0.035" rpy="0 -1.57 0"/>
-    <xacro:profile_channel parent="base_link" child="back_left_side_support_profile_channel"    profile_mass="0.045" profile_length="${Chassis_side_profile_length}" profile_width="${Chassis_profile_size}"  profile_height="${Chassis_profile_size}"  xyz="-0.290   0.290  0.035"  rpy="0 -1.57 0"/>
-    <xacro:profile_channel parent="base_link" child="back_right_side_support_profile_channel"   profile_mass="0.045" profile_length="${Chassis_side_profile_length}" profile_width="${Chassis_profile_size}"  profile_height="${Chassis_profile_size}"  xyz="-0.290  -0.290  0.035"  rpy="0 -1.57 0"/>
+    <xacro:profile_channel parent="base_link" child="left_bottom_motor_support_profile_channel" profile_mass="0.2425" profile_length="${motor_support_profile_length}" profile_width="${Chassis_profile_size}"  profile_height="${Chassis_profile_size}"  xyz="-0.0475  0.205   0.00"   rpy="0 0 0" />
+    <xacro:profile_channel parent="base_link" child="right_bottom_motor_support_profile_channel"  profile_mass="0.2425" profile_length="${motor_support_profile_length}" profile_width="${Chassis_profile_size}"  profile_height="${Chassis_profile_size}"  xyz=" 0.0475 -0.205   0.00"   rpy="0 0 0" />
+    <xacro:profile_channel parent="base_link" child="front_top_profile_channel" profile_mass="0.28" profile_length="${Chassis_profile_length}" profile_width="${Chassis_profile_size}"  profile_height="${Chassis_profile_size}"  xyz=" 0.290   0.00  0.130"   rpy="0 0 -1.57" />
+    <xacro:profile_channel parent="base_link" child="back_top_profile_channel"  profile_mass="0.28" profile_length="${Chassis_profile_length}" profile_width="${Chassis_profile_size}"  profile_height="${Chassis_profile_size}"  xyz="-0.290   0.00  0.130"    rpy="0 0 -1.57" />
+    <xacro:profile_channel parent="base_link" child="left_top_profile_channel"  profile_mass="0.28" profile_length="${Chassis_profile_length}" profile_width="${Chassis_profile_size}"  profile_height="${Chassis_profile_size}"  xyz=" 0.0     0.290 0.130"  rpy="0 0 0" />
+    <xacro:profile_channel parent="base_link" child="right_top_profile_channel" profile_mass="0.28" profile_length="${Chassis_profile_length}" profile_width="${Chassis_profile_size}"  profile_height="${Chassis_profile_size}"  xyz=" 0.0    -0.290 0.130"  rpy="0 0 0" />
+    <xacro:profile_channel parent="base_link" child="front_top_motor_support_profile_channel"    profile_mass="0.2425" profile_length="${motor_support_profile_length}" profile_width="${Chassis_profile_size}"  profile_height="${Chassis_profile_size}"  xyz=" 0.205   0.0475  0.130"  rpy="0 0 -1.57"/>
+    <xacro:profile_channel parent="base_link" child="back_top_motor_support_profile_channel"     profile_mass="0.2425" profile_length="${motor_support_profile_length}" profile_width="${Chassis_profile_size}"  profile_height="${Chassis_profile_size}"  xyz="-0.205  -0.0475  0.130"  rpy="0 0 -1.57"/>
+    <xacro:profile_channel parent="base_link" child="left_top_motor_support_profile_channel"     profile_mass="0.2425" profile_length="${motor_support_profile_length}" profile_width="${Chassis_profile_size}"  profile_height="${Chassis_profile_size}"  xyz="-0.0475  0.205   0.130"  rpy="0 0 0"/>
+    <xacro:profile_channel parent="base_link" child="right_top_motor_support_profile_channel"    profile_mass="0.2425" profile_length="${motor_support_profile_length}" profile_width="${Chassis_profile_size}"  profile_height="${Chassis_profile_size}"  xyz=" 0.0475 -0.205   0.130"  rpy="0 0 0"/>
+    <xacro:profile_channel parent="base_link" child="front_left_side_support_profile_channel"   profile_mass="0.045" profile_length="${Chassis_side_profile_length}" profile_width="${Chassis_profile_size}"  profile_height="${Chassis_profile_size}"  xyz=" 0.290   0.290  0.065" rpy="0 -1.57 0"/>
+    <xacro:profile_channel parent="base_link" child="front_right_side_support_profile_channel"  profile_mass="0.045" profile_length="${Chassis_side_profile_length}" profile_width="${Chassis_profile_size}"  profile_height="${Chassis_profile_size}"  xyz=" 0.290  -0.290  0.065" rpy="0 -1.57 0"/>
+    <xacro:profile_channel parent="base_link" child="back_left_side_support_profile_channel"    profile_mass="0.045" profile_length="${Chassis_side_profile_length}" profile_width="${Chassis_profile_size}"  profile_height="${Chassis_profile_size}"  xyz="-0.290   0.290  0.065"  rpy="0 -1.57 0"/>
+    <xacro:profile_channel parent="base_link" child="back_right_side_support_profile_channel"   profile_mass="0.045" profile_length="${Chassis_side_profile_length}" profile_width="${Chassis_profile_size}"  profile_height="${Chassis_profile_size}"  xyz="-0.290  -0.290  0.065"  rpy="0 -1.57 0"/>
     <!-- Bot Front Marker -->
-    <xacro:profile_channel parent="base_link" child="Bot_Front_Marker_profile_channel"   profile_mass="0.001" profile_length="${Chassis_side_profile_length}" profile_width="${Chassis_profile_size}"  profile_height="${Chassis_profile_size}"  xyz="0.290  0  0.105"  rpy="0 -1.57 0"/>
-    <!-- Omni Wheels-->
-    <xacro:omni_wheel parent="base_link" child="front_left"  xyz=" 0.255   0.205 0.035"  rpy=" 0.0   1.57 0.0 "/>
-    <xacro:omni_wheel parent="base_link" child="back_right"   xyz="-0.255  -0.205 0.035"  rpy=" 0.0  -1.57 0.0"/>
-    <xacro:omni_wheel parent="base_link" child="back_left"   xyz="-0.205  0.255 0.035"   rpy="-1.57  0    0.0"/>
-    <xacro:omni_wheel parent="base_link" child="front_right"  xyz=" 0.205 -0.255 0.035"   rpy=" 1.57  0    0.0"/>
+    <!-- <xacro:profile_channel parent="base_link" child="Bot_Front_Marker_profile_channel"   profile_mass="0.001" profile_length="${Chassis_side_profile_length}" profile_width="${Chassis_profile_size}"  profile_height="${Chassis_profile_size}"  xyz="0.290  0  0.105"  rpy="0 -1.57 0"/> -->
     <!-- Wheels-->
-    <!--<xacro:wheel parent="base_link" child="front_left"  xyz=" 0.245   0.205 0.035"  rpy=" 0.0   1.57 0.0 "/>
-    <xacro:wheel parent="base_link" child="back_right"   xyz="-0.245  -0.205 0.035"  rpy=" 0.0  -1.57 0.0"/>
-    <xacro:wheel parent="base_link" child="back_left"   xyz="-0.205  0.245 0.035"   rpy="-1.57  0    0.0"/>
-    <xacro:wheel parent="base_link" child="front_right"  xyz=" 0.205 -0.245 0.035"   rpy=" 1.57  0    0.0"/>-->
+    <xacro:if value="$(arg use_omni_wheel)">
+        <!-- Omni Wheels -->
+        <xacro:include filename="omni_wheel.xacro"/>
+        <xacro:omni_wheel parent="base_link" child="front_left"  xyz=" 0.255   0.205 0.035"  rpy=" 0.0   1.57 0.0 "/>
+        <xacro:omni_wheel parent="base_link" child="back_right"   xyz="-0.255  -0.205 0.035"  rpy=" 0.0  -1.57 0.0"/>
+        <xacro:omni_wheel parent="base_link" child="back_left"   xyz="-0.205  0.255 0.035"   rpy="-1.57  0    0.0"/>
+        <xacro:omni_wheel parent="base_link" child="front_right"  xyz=" 0.205 -0.255 0.035"   rpy=" 1.57  0    0.0"/>
+    </xacro:if>
+    <xacro:unless value="$(arg use_omni_wheel)">
+        <!--Normal Wheels-->
+        <xacro:include filename="wheel.xacro"/>
+        <xacro:wheel parent="base_link" child="front_left"  xyz=" 0.245   0.205 0.035"  rpy=" 0.0   1.57 0.0 "/>
+        <xacro:wheel parent="base_link" child="back_right"   xyz="-0.245  -0.205 0.035"  rpy=" 0.0  -1.57 0.0"/>
+        <xacro:wheel parent="base_link" child="back_left"   xyz="-0.205  0.245 0.035"   rpy="-1.57  0    0.0"/>
+        <xacro:wheel parent="base_link" child="front_right"  xyz=" 0.205 -0.245 0.035"   rpy=" 1.57  0    0.0"/>
+    </xacro:unless>
 </robot>
