Commit message: Add files via upload

File: description/arm.xacro (robot description, xacro)
@@ -2,328 +2,177 @@
 <robot xmlns:xacro="http://www.ros.org/wiki/xacro">
     <xacro:include filename="inertial_macros.xacro"/>
-    <link name="right_sholder">
-        <visual>
-            <origin xyz="0.0 0.0 0.0" rpy="0.0 0.0 3.14"/>
-            <geometry>
-                <mesh filename="file://$(find project_eva)/meshes/EVA/Arm/sholder.STL"/>
-            </geometry>
-            <material name="Top">
-                <color rgba="${48/255} ${104/255} ${68/255} 1.0"/>
-            </material>
-        </visual>
-        <collision>
-            <origin xyz="0.0 -0.035 0.0" rpy="0.0 0.0 0.0"/>
-            <geometry>
-                <box size="0.070 0.080 0.050 "/>
-            </geometry>
-        </collision>
-        <xacro:inertial_box mass="0.3" x="0.070" y="0.080" z="0.050">
-            <origin xyz="0.0 -0.035 0.0" rpy="0.0 0.0 0.0"/>
-        </xacro:inertial_box>
-    </link>
-    <joint name="right_arm_joint" type="revolute">
-        <axis xyz="0 1 0"/>
-        <limit effort="0.1" lower="-2.0" upper="0.51" velocity="0.2"/>
-        <origin xyz="0 -0.118 0.457" rpy="3.14 3.14 3.14"/>
-        <parent link="body" />
-        <child link="right_sholder" />
-    </joint>
-    <link name="right_upper_biceps">
-        <visual>
-            <origin xyz="0.0 0.0 0.0" rpy="0.0 0.0 0.0"/>
-            <geometry>
-                <mesh filename="file://$(find project_eva)/meshes/EVA/Arm/upper_biceps.STL"/>
-            </geometry>
-            <material name="skin">
-                <color rgba="${255/255} ${219/255} ${184/255} 1.0"/>
-            </material>
-        </visual>
-        <collision>
-            <origin xyz="0.0 0.0 -0.0450" rpy="0.0 0.0 0.0"/>
-            <geometry>
-                <cylinder radius="0.038" length="0.090"/>
-            </geometry>
-        </collision>
-        <xacro:inertial_cylinder mass="0.03" radius="0.038"  length="0.090" >
-            <origin xyz="0.0 0.0 -0.0450" rpy="0.0 0.0 0.0"/>
-        </xacro:inertial_cylinder>
-    </link>
-    <joint name="right_sholder_joint" type="revolute">
-        <axis xyz="1 0 0"/>
-        <limit effort="0.1" lower="-2.09" upper="0" velocity="0.2"/>
-        <origin xyz="0 -0.040 0" rpy="0 0 0" />
-        <parent link="right_sholder" />
-        <child link="right_upper_biceps" />
-    </joint>
-    <link name="right_lower_biceps">
-        <visual>
-            <origin xyz="0.0 0.0 0.0" rpy="-0.07 0 0"/>
-            <geometry>
-                <mesh filename="file://$(find project_eva)/meshes/EVA/Arm/lower_biceps.STL"/>
-            </geometry>
-            <material name="skin">
-                <color rgba="${255/255} ${219/255} ${184/255} 1.0"/>
-            </material>
-        </visual>
-        <collision>
-            <origin xyz="0.0 0.0 -0.0915" rpy="0.0 0.0 0.0"/>
-            <geometry>
-                <cylinder radius="0.038" length="0.1830"/>
-            </geometry>
-        </collision>
-        <xacro:inertial_cylinder mass="0.03" radius="0.038" length="0.1830">
-            <origin xyz="0.0 0.0 -0.0915" rpy="0.0 0.0 0.0"/>
-        </xacro:inertial_cylinder>
-    </link>
-    <joint name="right_biceps_joint" type="revolute">
-        <axis xyz="0 0 1"/>
-        <limit effort="0.1" lower="0" upper="1.57" velocity="0.2"/>
-        <origin xyz="0 0 -0.090" rpy="0 0 0" />
-        <parent link="right_upper_biceps" />
-        <child link="right_lower_biceps" />
-    </joint>
-    <link name="right_elbow">
-        <visual>
-            <origin xyz="0.0 -0.0015 0.0" rpy="0 0 0"/>
-            <geometry>
-                <mesh filename="file://$(find project_eva)/meshes/EVA/Arm/elbow.STL"/>
-            </geometry>
-            <material name="skin">
-                <color rgba="${255/255} ${219/255} ${184/255} 1.0"/>
-            </material>
-        </visual>
-        <collision>
-            <origin xyz="0.0 0.0 -0.02175" rpy="0.0 0.0 0.0"/>
-            <geometry>
-                <cylinder radius="0.038" length="0.0435"/>
-            </geometry>
-        </collision>
-        <xacro:inertial_cylinder mass="0.03" radius="0.038" length="0.0435" >
-            <origin xyz="0.0 0.0 0.02175" rpy="0.0 0.0 0.0"/>
-        </xacro:inertial_cylinder>
-    </link>
-    <joint name="right_elbow_joint" type="revolute">
-        <axis xyz="0 1 0"/>
-        <limit effort="0.1" lower="0" upper="-2.05" velocity="0.2"/>
-        <origin xyz="0 0 -0.1830" rpy="0 0 0" />
-        <parent link="right_lower_biceps" />
-        <child link="right_elbow" />
-    </joint>
-    <link name="right_wrist">
-        <visual>
-            <origin xyz="0.0 -0.003 0.0440" rpy="0.0 0.0 0.0"/>
-            <geometry>
-                <mesh filename="file://$(find project_eva)/meshes/EVA/Arm/wrist.STL"/>
-            </geometry>
-            <material name="skin">
-                <color rgba="${255/255} ${219/255} ${184/255} 1.0"/>
-            </material>
-        </visual>
-        <collision>
-            <origin xyz="0.0 0.0 -0.0827" rpy="0.0 0.0 0.0"/>
-            <geometry>
-                <cylinder radius="0.030" length="0.1654"/>
-            </geometry>
-        </collision>
-        <xacro:inertial_cylinder mass="0.03" radius="0.030" length="0.1554" >
-            <origin xyz="0 0 0" rpy="0 0 0"/>
-        </xacro:inertial_cylinder>
-    </link>
-    <joint name="right_wrist_joint" type="revolute">
-        <axis xyz="0 0 1"/>
-        <limit effort="0.1" lower="-1.57" upper="1.57" velocity="0.2"/>
-        <origin xyz="0 0 -0.0435" rpy="0 0 0" />
-        <parent link="right_elbow" />
-        <child link="right_wrist" />
-    </joint>
-    <link name="right_hand">
-        <visual>
-            <origin xyz="0.0 0.0 0.0" rpy="0 0 1.57"/>
-            <geometry>
-                <mesh filename="file://$(find project_eva)/meshes/EVA/Arm/hand.STL"/>
-            </geometry>
-            <material name="skin">
-                <color rgba="${255/255} ${219/255} ${184/255} 1.0"/>
-            </material>
-        </visual>
-        <collision>
-            <origin xyz="0.0 0.0 -0.045" rpy="0.0 0.0 0.0"/>
-            <geometry>
-                <box size="0.060 0.030 0.090"/>
-            </geometry>
-        </collision>
-        <xacro:inertial_box mass="0.3" x="0.070" y="0.080" z="0.050">
-            <origin xyz="0 0 0" rpy="0 0 0"/>
-        </xacro:inertial_box>
-    </link>
-    <joint name="right_hand_joint" type="revolute">
-        <axis xyz="1 0 0"/>
-        <limit effort="0.1" lower="-0.6" upper="1.10" velocity="0.2"/>
-        <origin xyz="0 0.002 -0.167" rpy="0 0 0" />
-        <parent link="right_wrist" />
-        <child link="right_hand" />
-    </joint>
-<!--          Left arm        -->
-    <link name="left_sholder">
-        <visual>
-            <origin xyz="0.0 0.0 0.0" rpy="0.0 0.0 0"/>
-            <geometry>
-                <mesh filename="file://$(find project_eva)/meshes/EVA/Arm/sholder.STL"/>
-            </geometry>
-            <material name="Top">
-                <color rgba="${48/255} ${104/255} ${68/255} 1.0"/>
-            </material>
-        </visual>
-        <collision>
-            <origin xyz="0.0 0.035 0.0" rpy="0.0 0.0 0.0"/>
-            <geometry>
-                <box size="0.070 0.080 0.050 "/>
-            </geometry>
-        </collision>
-        <xacro:inertial_box mass="0.3" x="0.070" y="0.080" z="0.050">
-            <origin xyz="0.0 0.035 0.0" rpy="0.0 0.0 0.0"/>
-        </xacro:inertial_box>
-    </link>
-    <joint name="left_arm_joint" type="revolute">
-        <axis xyz="0 1 0"/>
-        <limit effort="0.1" lower="-2.0" upper="0.51" velocity="0.2"/>
-        <origin xyz="0 0.118 0.457" rpy="0 0 0"/>
-        <parent link="body" />
-        <child link="left_sholder" />
-    </joint>
-    <link name="left_upper_biceps">
-        <visual>
-            <origin xyz="0.0 0.0 0.0" rpy="0.0 0.0 0.0"/>
-            <geometry>
-                <mesh filename="file://$(find project_eva)/meshes/EVA/Arm/upper_biceps.STL"/>
-            </geometry>
-            <material name="skin">
-                <color rgba="${255/255} ${219/255} ${184/255} 1.0"/>
-            </material>
-        </visual>
-        <collision>
-            <origin xyz="0.0 0.0 -0.0450" rpy="0.0 0.0 0.0"/>
-            <geometry>
-                <cylinder radius="0.038" length="0.090"/>
-            </geometry>
-        </collision>
-        <xacro:inertial_cylinder mass="0.03" radius="0.038"  length="0.090" >
-            <origin xyz="0.0 0.0 -0.0450" rpy="0.0 0.0 0.0"/>
-        </xacro:inertial_cylinder>
-    </link>
-    <joint name="left_sholder_joint" type="revolute">
-        <axis xyz="1 0 0"/>
-        <limit effort="0.1" lower="0" upper="2.09" velocity="0.2"/>
-        <origin xyz="0 0.040 0" rpy="0 0 0" />
-        <parent link="left_sholder" />
-        <child link="left_upper_biceps" />
-    </joint>
-    <link name="left_lower_biceps">
-        <visual>
-            <origin xyz="0.0 0.0 0.0" rpy="-0.07 0 0"/>
-            <geometry>
-                <mesh filename="file://$(find project_eva)/meshes/EVA/Arm/lower_biceps.STL"/>
-            </geometry>
-            <material name="skin">
-                <color rgba="${255/255} ${219/255} ${184/255} 1.0"/>
-            </material>
-        </visual>
-        <collision>
-            <origin xyz="0.0 0.0 -0.0915" rpy="0.0 0.0 0.0"/>
-            <geometry>
-                <cylinder radius="0.038" length="0.1830"/>
-            </geometry>
-        </collision>
-        <xacro:inertial_cylinder mass="0.03" radius="0.038" length="0.1830">
-            <origin xyz="0.0 0.0 -0.0915" rpy="0.0 0.0 0.0"/>
-        </xacro:inertial_cylinder>
-    </link>
-    <joint name="left_biceps_joint" type="revolute">
-        <axis xyz="0 0 1"/>
-        <limit effort="0.1" lower="-1.57" upper="0" velocity="0.2"/>
-        <origin xyz="0 0 -0.090" rpy="0 0 0" />
-        <parent link="left_upper_biceps" />
-        <child link="left_lower_biceps" />
-    </joint>
-    <link name="left_elbow">
-        <visual>
-            <origin xyz="0.0 -0.0015 0.0" rpy="0 0 0"/>
-            <geometry>
-                <mesh filename="file://$(find project_eva)/meshes/EVA/Arm/elbow.STL"/>
-            </geometry>
-            <material name="skin">
-                <color rgba="${255/255} ${219/255} ${184/255} 1.0"/>
-            </material>
-        </visual>
-        <collision>
-            <origin xyz="0.0 0.0 -0.02175" rpy="0.0 0.0 0.0"/>
-            <geometry>
-                <cylinder radius="0.038" length="0.0435"/>
-            </geometry>
-        </collision>
-        <xacro:inertial_cylinder mass="0.03" radius="0.038" length="0.0435" >
-            <origin xyz="0.0 0.0 0.02175" rpy="0.0 0.0 0.0"/>
-        </xacro:inertial_cylinder>
-    </link>
-    <joint name="left_elbow_joint" type="revolute">
-        <axis xyz="0 1 0"/>
-        <limit effort="0.1" lower="0" upper="-2.05" velocity="0.2"/>
-        <origin xyz="0 0 -0.1830" rpy="0 0 0" />
-        <parent link="left_lower_biceps" />
-        <child link="left_elbow" />
-    </joint>
-    <link name="left_wrist">
-        <visual>
-            <origin xyz="0.0 -0.003 0.0440" rpy="0.0 0.0 0.0"/>
-            <geometry>
-                <mesh filename="file://$(find project_eva)/meshes/EVA/Arm/wrist.STL"/>
-            </geometry>
-            <material name="skin">
-                <color rgba="${255/255} ${219/255} ${184/255} 1.0"/>
-            </material>
-        </visual>
-        <collision>
-            <origin xyz="0.0 0.0 -0.0827" rpy="0.0 0.0 0.0"/>
-            <geometry>
-                <cylinder radius="0.030" length="0.1654"/>
-            </geometry>
-        </collision>
-        <xacro:inertial_cylinder mass="0.03" radius="0.030" length="0.1554" >
-            <origin xyz="0 0 0" rpy="0 0 0"/>
-        </xacro:inertial_cylinder>
-    </link>
-    <joint name="left_wrist_joint" type="revolute">
-        <axis xyz="0 0 1"/>
-        <limit effort="0.1" lower="-1.57" upper="1.57" velocity="0.2"/>
-        <origin xyz="0 0 -0.0435" rpy="0 0 0" />
-        <parent link="left_elbow" />
-        <child link="left_wrist" />
-    </joint>
-    <link name="left_hand">
-        <visual>
-            <origin xyz="0.0 0.0 0.0" rpy="0 0 1.57"/>
-            <geometry>
-                <mesh filename="file://$(find project_eva)/meshes/EVA/Arm/hand.STL"/>
-            </geometry>
-            <material name="skin">
-                <color rgba="${255/255} ${219/255} ${184/255} 1.0"/>
-            </material>
-        </visual>
-        <collision>
-            <origin xyz="0.0 0.0 -0.045" rpy="0.0 0.0 0.0"/>
-            <geometry>
-                <box size="0.060 0.030 0.090"/>
-            </geometry>
-        </collision>
-        <xacro:inertial_box mass="0.3" x="0.070" y="0.080" z="0.050">
-            <origin xyz="0 0 0" rpy="0 0 0"/>
-        </xacro:inertial_box>
-    </link>
-    <joint name="left_hand_joint" type="revolute">
-        <axis xyz="1 0 0"/>
-        <limit effort="0.1" lower="-1.10" upper="0.6" velocity="0.2"/>
-        <origin xyz="0 0.002 -0.167" rpy="0 0 0" />
-        <parent link="left_wrist" />
-        <child link="left_hand" />
-    </joint>
+    <xacro:macro name="sholder" params="parent child v_rpy c_xyz o_xyz o_rpy">
+        <link name="${child}_sholder">
+            <visual>
+                <origin xyz="0.0 0.0 0.0" rpy="${v_rpy}"/>
+                <geometry>
+                    <mesh filename="file://$(find project_eva)/meshes/EVA/Arm/sholder.STL"/>
+                </geometry>
+                <material name="Top">
+                    <color rgba="${48/255} ${104/255} ${68/255} 1.0"/>
+                </material>
+            </visual>
+            <collision>
+                <origin xyz="${c_xyz}" rpy="0.0 0.0 0.0"/>
+                <geometry>
+                    <box size="0.070 0.080 0.050 "/>
+                </geometry>
+            </collision>
+            <xacro:inertial_box mass="0.3" x="0.070" y="0.080" z="0.050">
+                <origin xyz="${c_xyz}" rpy="0.0 0.0 0.0"/>
+            </xacro:inertial_box>
+        </link>
+        <joint name="${child}_arm_joint" type="revolute">
+            <axis xyz="0 1 0"/>
+            <limit effort="0.1" lower="-2.0" upper="0.51" velocity="0.2"/>
+            <origin xyz="${o_xyz}" rpy="${o_rpy}"/>
+            <parent link="${parent}" />
+            <child link="${child}_sholder" />
+        </joint>
+    </xacro:macro>
+    <xacro:macro name="upper_biceps" params="side lower upper o_xyz">
+        <link name="${side}_upper_biceps">
+            <visual>
+                <origin xyz="0.0 0.0 0.0" rpy="0.0 0.0 0.0"/>
+                <geometry>
+                    <mesh filename="file://$(find project_eva)/meshes/EVA/Arm/upper_biceps.STL"/>
+                </geometry>
+                <material name="skin">
+                    <color rgba="${255/255} ${219/255} ${184/255} 1.0"/>
+                </material>
+            </visual>
+            <collision>
+                <origin xyz="0.0 0.0 -0.0450" rpy="0.0 0.0 0.0"/>
+                <geometry>
+                    <cylinder radius="0.038" length="0.090"/>
+                </geometry>
+            </collision>
+            <xacro:inertial_cylinder mass="0.03" radius="0.038"  length="0.090" >
+                <origin xyz="0.0 0.0 -0.0450" rpy="0.0 0.0 0.0"/>
+            </xacro:inertial_cylinder>
+        </link>
+        <joint name="${side}_sholder_joint" type="revolute">
+            <axis xyz="1 0 0"/>
+            <limit effort="0.1" lower="${lower}" upper="${upper}" velocity="0.2"/>
+            <origin xyz="${o_xyz}" rpy="0 0 0" />
+            <parent link="${side}_sholder" />
+            <child link="${side}_upper_biceps" />
+        </joint>
+    </xacro:macro>
+    <xacro:macro name="lower_biceps" params="side lower upper">
+        <link name="${side}_lower_biceps">
+            <visual>
+                <origin xyz="0.0 0.0 0.0" rpy="-0.07 0 0"/>
+                <geometry>
+                    <mesh filename="file://$(find project_eva)/meshes/EVA/Arm/lower_biceps.STL"/>
+                </geometry>
+                <material name="skin">
+                    <color rgba="${255/255} ${219/255} ${184/255} 1.0"/>
+                </material>
+            </visual>
+            <collision>
+                <origin xyz="0.0 0.0 -0.0915" rpy="0.0 0.0 0.0"/>
+                <geometry>
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
File: description/body.xacro (robot description, xacro)
@@ -97,5 +97,5 @@
                 </geometry>
         </collision>
-        <xacro:inertial_cylinder mass="${wheel_mass}" length="${wheel_thickness}" radius="${wheel_radius}">
+        <xacro:inertial_cylinder mass="0.02" length="0.1" radius="0.1">
             <origin xyz="0 0 0" rpy="0 0 0"/>
         </xacro:inertial_cylinder>

File: description/robot.urdf.xacro (robot description, xacro)
@@ -2,9 +2,6 @@
 <robot xmlns:xacro="http://www.ros.org/wiki/xacro"  name="robot">
     <xacro:arg name="use_omni_wheel" default="false"/>
+    <xacro:arg name="use_arm" default="false"/>
     <xacro:include filename="robot_core.xacro"/>
-    <xacro:include filename="arm.xacro"/>
-    <xacro:include filename="body.xacro"/>
-    <xacro:include filename="leg.xacro"/>
-    <xacro:include filename="realsense.xacro"/>
     <!-- <xacro:include filename="gazebo_control.xacro"/> -->
     <!-- <xacro:include filename="ros2_control.xacro"/> -->
