Commit message: Add files via upload

File: description/robot_core.xacro (robot description, xacro)
@@ -3,8 +3,6 @@
     <xacro:include filename="profile_channel.xacro"/>
     <!-- Base Link -->
-    <link name="base_link">
-    </link>
-    <link name="EVA_base_link">
-    </link>
+    <link name="base_link"></link>
+    <link name="EVA_base_link"></link>
     <joint name="base_joint" type="fixed">
         <parent link="base_link"/>
@@ -12,47 +10,68 @@
         <origin xyz="0 0 0.140" rpy="0 0 0" />
     </joint>
-    <!-- Chassis profile Channels -->
-    <xacro:property name="Chassis_profile_size" value="0.02"/>
-    <xacro:property name="Chassis_profile_length" value="0.560"/>
-    <xacro:property name="Chassis_side_profile_length" value="0.150"/>
-    <xacro:property name="motor_support_profile_length" value="0.485"/>
-    <xacro:profile_channel parent="base_link" child="front_bottom_profile_channel" profile_mass="0.28" profile_length="${Chassis_profile_length}" profile_width="${Chassis_profile_size}"  profile_height="${Chassis_profile_size}"  xyz=" 0.290   0.00  0.00"   rpy="0 0 -1.57" />
-    <xacro:profile_channel parent="base_link" child="back_bottom_profile_channel"  profile_mass="0.28" profile_length="${Chassis_profile_length}" profile_width="${Chassis_profile_size}"  profile_height="${Chassis_profile_size}"  xyz="-0.290   0.00  0.00"    rpy="0 0 -1.57" />
-    <xacro:profile_channel parent="base_link" child="left_bottom_profile_channel"  profile_mass="0.28" profile_length="${Chassis_profile_length}" profile_width="${Chassis_profile_size}"  profile_height="${Chassis_profile_size}"  xyz=" 0.0     0.290 0.00"  rpy="0 0 0" />
-    <xacro:profile_channel parent="base_link" child="right_bottom_profile_channel" profile_mass="0.28" profile_length="${Chassis_profile_length}" profile_width="${Chassis_profile_size}"  profile_height="${Chassis_profile_size}"  xyz=" 0.0    -0.290 0.00"  rpy="0 0 0" />
-    <xacro:profile_channel parent="base_link" child="front_bottom_motor_support_profile_channel" profile_mass="0.2425" profile_length="${motor_support_profile_length}" profile_width="${Chassis_profile_size}"  profile_height="${Chassis_profile_size}"  xyz=" 0.205   0.0475  0.00"   rpy="0 0 -1.57"/>
-    <xacro:profile_channel parent="base_link" child="back_bottom_motor_support_profile_channel"  profile_mass="0.2425" profile_length="${motor_support_profile_length}" profile_width="${Chassis_profile_size}"  profile_height="${Chassis_profile_size}"  xyz="-0.205  -0.0475  0.00"   rpy="0 0 -1.57"/>
-    <xacro:profile_channel parent="base_link" child="left_bottom_motor_support_profile_channel" profile_mass="0.2425" profile_length="${motor_support_profile_length}" profile_width="${Chassis_profile_size}"  profile_height="${Chassis_profile_size}"  xyz="-0.0475  0.205   0.00"   rpy="0 0 0" />
-    <xacro:profile_channel parent="base_link" child="right_bottom_motor_support_profile_channel"  profile_mass="0.2425" profile_length="${motor_support_profile_length}" profile_width="${Chassis_profile_size}"  profile_height="${Chassis_profile_size}"  xyz=" 0.0475 -0.205   0.00"   rpy="0 0 0" />
-    <xacro:profile_channel parent="base_link" child="front_top_profile_channel" profile_mass="0.28" profile_length="${Chassis_profile_length}" profile_width="${Chassis_profile_size}"  profile_height="${Chassis_profile_size}"  xyz=" 0.290   0.00  0.130"   rpy="0 0 -1.57" />
-    <xacro:profile_channel parent="base_link" child="back_top_profile_channel"  profile_mass="0.28" profile_length="${Chassis_profile_length}" profile_width="${Chassis_profile_size}"  profile_height="${Chassis_profile_size}"  xyz="-0.290   0.00  0.130"    rpy="0 0 -1.57" />
-    <xacro:profile_channel parent="base_link" child="left_top_profile_channel"  profile_mass="0.28" profile_length="${Chassis_profile_length}" profile_width="${Chassis_profile_size}"  profile_height="${Chassis_profile_size}"  xyz=" 0.0     0.290 0.130"  rpy="0 0 0" />
-    <xacro:profile_channel parent="base_link" child="right_top_profile_channel" profile_mass="0.28" profile_length="${Chassis_profile_length}" profile_width="${Chassis_profile_size}"  profile_height="${Chassis_profile_size}"  xyz=" 0.0    -0.290 0.130"  rpy="0 0 0" />
-    <xacro:profile_channel parent="base_link" child="front_top_motor_support_profile_channel"    profile_mass="0.2425" profile_length="${motor_support_profile_length}" profile_width="${Chassis_profile_size}"  profile_height="${Chassis_profile_size}"  xyz=" 0.205   0.0475  0.130"  rpy="0 0 -1.57"/>
-    <xacro:profile_channel parent="base_link" child="back_top_motor_support_profile_channel"     profile_mass="0.2425" profile_length="${motor_support_profile_length}" profile_width="${Chassis_profile_size}"  profile_height="${Chassis_profile_size}"  xyz="-0.205  -0.0475  0.130"  rpy="0 0 -1.57"/>
-    <xacro:profile_channel parent="base_link" child="left_top_motor_support_profile_channel"     profile_mass="0.2425" profile_length="${motor_support_profile_length}" profile_width="${Chassis_profile_size}"  profile_height="${Chassis_profile_size}"  xyz="-0.0475  0.205   0.130"  rpy="0 0 0"/>
-    <xacro:profile_channel parent="base_link" child="right_top_motor_support_profile_channel"    profile_mass="0.2425" profile_length="${motor_support_profile_length}" profile_width="${Chassis_profile_size}"  profile_height="${Chassis_profile_size}"  xyz=" 0.0475 -0.205   0.130"  rpy="0 0 0"/>
-    <xacro:profile_channel parent="base_link" child="front_left_side_support_profile_channel"   profile_mass="0.045" profile_length="${Chassis_side_profile_length}" profile_width="${Chassis_profile_size}"  profile_height="${Chassis_profile_size}"  xyz=" 0.290   0.290  0.065" rpy="0 -1.57 0"/>
-    <xacro:profile_channel parent="base_link" child="front_right_side_support_profile_channel"  profile_mass="0.045" profile_length="${Chassis_side_profile_length}" profile_width="${Chassis_profile_size}"  profile_height="${Chassis_profile_size}"  xyz=" 0.290  -0.290  0.065" rpy="0 -1.57 0"/>
-    <xacro:profile_channel parent="base_link" child="back_left_side_support_profile_channel"    profile_mass="0.045" profile_length="${Chassis_side_profile_length}" profile_width="${Chassis_profile_size}"  profile_height="${Chassis_profile_size}"  xyz="-0.290   0.290  0.065"  rpy="0 -1.57 0"/>
-    <xacro:profile_channel parent="base_link" child="back_right_side_support_profile_channel"   profile_mass="0.045" profile_length="${Chassis_side_profile_length}" profile_width="${Chassis_profile_size}"  profile_height="${Chassis_profile_size}"  xyz="-0.290  -0.290  0.065"  rpy="0 -1.57 0"/>
-    <!-- Bot Front Marker -->
-    <!-- <xacro:profile_channel parent="base_link" child="Bot_Front_Marker_profile_channel"   profile_mass="0.001" profile_length="${Chassis_side_profile_length}" profile_width="${Chassis_profile_size}"  profile_height="${Chassis_profile_size}"  xyz="0.290  0  0.105"  rpy="0 -1.57 0"/> -->
-    <!-- Wheels-->
-    <xacro:if value="$(arg use_omni_wheel)">
-        <!-- Omni Wheels -->
-        <xacro:include filename="omni_wheel.xacro"/>
-        <xacro:omni_wheel parent="base_link" child="front_left"  xyz=" 0.255   0.205 0.035"  rpy=" 0.0   1.57 0.0 "/>
-        <xacro:omni_wheel parent="base_link" child="back_right"   xyz="-0.255  -0.205 0.035"  rpy=" 0.0  -1.57 0.0"/>
-        <xacro:omni_wheel parent="base_link" child="back_left"   xyz="-0.205  0.255 0.035"   rpy="-1.57  0    0.0"/>
-        <xacro:omni_wheel parent="base_link" child="front_right"  xyz=" 0.205 -0.255 0.035"   rpy=" 1.57  0    0.0"/>
+    <xacro:if value="$(arg use_drive)">
+        <!-- Chassis profile Channels -->
+        <xacro:property name="Chassis_profile_size" value="0.02"/>
+        <xacro:property name="Chassis_profile_length" value="0.560"/>
+        <xacro:property name="Chassis_side_profile_length" value="0.150"/>
+        <xacro:property name="motor_support_profile_length" value="0.485"/>
+        <xacro:profile_channel parent="base_link" child="front_bottom_profile_channel" profile_mass="0.28" profile_length="${Chassis_profile_length}" profile_width="${Chassis_profile_size}"  profile_height="${Chassis_profile_size}"  xyz=" 0.290   0.00  0.00"   rpy="0 0 -1.57" />
+        <xacro:profile_channel parent="base_link" child="back_bottom_profile_channel"  profile_mass="0.28" profile_length="${Chassis_profile_length}" profile_width="${Chassis_profile_size}"  profile_height="${Chassis_profile_size}"  xyz="-0.290   0.00  0.00"    rpy="0 0 -1.57" />
+        <xacro:profile_channel parent="base_link" child="left_bottom_profile_channel"  profile_mass="0.28" profile_length="${Chassis_profile_length}" profile_width="${Chassis_profile_size}"  profile_height="${Chassis_profile_size}"  xyz=" 0.0     0.290 0.00"  rpy="0 0 0" />
+        <xacro:profile_channel parent="base_link" child="right_bottom_profile_channel" profile_mass="0.28" profile_length="${Chassis_profile_length}" profile_width="${Chassis_profile_size}"  profile_height="${Chassis_profile_size}"  xyz=" 0.0    -0.290 0.00"  rpy="0 0 0" />
+        <xacro:profile_channel parent="base_link" child="front_bottom_motor_support_profile_channel" profile_mass="0.2425" profile_length="${motor_support_profile_length}" profile_width="${Chassis_profile_size}"  profile_height="${Chassis_profile_size}"  xyz=" 0.205   0.0475  0.00"   rpy="0 0 -1.57"/>
+        <xacro:profile_channel parent="base_link" child="back_bottom_motor_support_profile_channel"  profile_mass="0.2425" profile_length="${motor_support_profile_length}" profile_width="${Chassis_profile_size}"  profile_height="${Chassis_profile_size}"  xyz="-0.205  -0.0475  0.00"   rpy="0 0 -1.57"/>
+        <xacro:profile_channel parent="base_link" child="left_bottom_motor_support_profile_channel" profile_mass="0.2425" profile_length="${motor_support_profile_length}" profile_width="${Chassis_profile_size}"  profile_height="${Chassis_profile_size}"  xyz="-0.0475  0.205   0.00"   rpy="0 0 0" />
+        <xacro:profile_channel parent="base_link" child="right_bottom_motor_support_profile_channel"  profile_mass="0.2425" profile_length="${motor_support_profile_length}" profile_width="${Chassis_profile_size}"  profile_height="${Chassis_profile_size}"  xyz=" 0.0475 -0.205   0.00"   rpy="0 0 0" />
+        <xacro:profile_channel parent="base_link" child="front_top_profile_channel" profile_mass="0.28" profile_length="${Chassis_profile_length}" profile_width="${Chassis_profile_size}"  profile_height="${Chassis_profile_size}"  xyz=" 0.290   0.00  0.130"   rpy="0 0 -1.57" />
+        <xacro:profile_channel parent="base_link" child="back_top_profile_channel"  profile_mass="0.28" profile_length="${Chassis_profile_length}" profile_width="${Chassis_profile_size}"  profile_height="${Chassis_profile_size}"  xyz="-0.290   0.00  0.130"    rpy="0 0 -1.57" />
+        <xacro:profile_channel parent="base_link" child="left_top_profile_channel"  profile_mass="0.28" profile_length="${Chassis_profile_length}" profile_width="${Chassis_profile_size}"  profile_height="${Chassis_profile_size}"  xyz=" 0.0     0.290 0.130"  rpy="0 0 0" />
+        <xacro:profile_channel parent="base_link" child="right_top_profile_channel" profile_mass="0.28" profile_length="${Chassis_profile_length}" profile_width="${Chassis_profile_size}"  profile_height="${Chassis_profile_size}"  xyz=" 0.0    -0.290 0.130"  rpy="0 0 0" />
+        <xacro:profile_channel parent="base_link" child="front_top_motor_support_profile_channel"    profile_mass="0.2425" profile_length="${motor_support_profile_length}" profile_width="${Chassis_profile_size}"  profile_height="${Chassis_profile_size}"  xyz=" 0.205   0.0475  0.130"  rpy="0 0 -1.57"/>
+        <xacro:profile_channel parent="base_link" child="back_top_motor_support_profile_channel"     profile_mass="0.2425" profile_length="${motor_support_profile_length}" profile_width="${Chassis_profile_size}"  profile_height="${Chassis_profile_size}"  xyz="-0.205  -0.0475  0.130"  rpy="0 0 -1.57"/>
+        <xacro:profile_channel parent="base_link" child="left_top_motor_support_profile_channel"     profile_mass="0.2425" profile_length="${motor_support_profile_length}" profile_width="${Chassis_profile_size}"  profile_height="${Chassis_profile_size}"  xyz="-0.0475  0.205   0.130"  rpy="0 0 0"/>
+        <xacro:profile_channel parent="base_link" child="right_top_motor_support_profile_channel"    profile_mass="0.2425" profile_length="${motor_support_profile_length}" profile_width="${Chassis_profile_size}"  profile_height="${Chassis_profile_size}"  xyz=" 0.0475 -0.205   0.130"  rpy="0 0 0"/>
+        <xacro:profile_channel parent="base_link" child="front_left_side_support_profile_channel"   profile_mass="0.045" profile_length="${Chassis_side_profile_length}" profile_width="${Chassis_profile_size}"  profile_height="${Chassis_profile_size}"  xyz=" 0.290   0.290  0.065" rpy="0 -1.57 0"/>
+        <xacro:profile_channel parent="base_link" child="front_right_side_support_profile_channel"  profile_mass="0.045" profile_length="${Chassis_side_profile_length}" profile_width="${Chassis_profile_size}"  profile_height="${Chassis_profile_size}"  xyz=" 0.290  -0.290  0.065" rpy="0 -1.57 0"/>
+        <xacro:profile_channel parent="base_link" child="back_left_side_support_profile_channel"    profile_mass="0.045" profile_length="${Chassis_side_profile_length}" profile_width="${Chassis_profile_size}"  profile_height="${Chassis_profile_size}"  xyz="-0.290   0.290  0.065"  rpy="0 -1.57 0"/>
+        <xacro:profile_channel parent="base_link" child="back_right_side_support_profile_channel"   profile_mass="0.045" profile_length="${Chassis_side_profile_length}" profile_width="${Chassis_profile_size}"  profile_height="${Chassis_profile_size}"  xyz="-0.290  -0.290  0.065"  rpy="0 -1.57 0"/>
+        <!-- Bot Front Marker -->
+        <!-- <xacro:profile_channel parent="base_link" child="Bot_Front_Marker_profile_channel"   profile_mass="0.001" profile_length="${Chassis_side_profile_length}" profile_width="${Chassis_profile_size}"  profile_height="${Chassis_profile_size}"  xyz="0.290  0  0.105"  rpy="0 -1.57 0"/> -->
+        <!-- Wheels-->
+        <xacro:if value="$(arg use_omni_wheel)">
+            <!-- Omni Wheels -->
+            <xacro:include filename="omni_wheel.xacro"/>
+            <xacro:omni_wheel parent="base_link" child="front_left"  xyz=" 0.255  0.205 0.035" rpy=" 0.0   1.57 0.0 "/>
+            <xacro:omni_wheel parent="base_link" child="back_right"  xyz="-0.255 -0.205 0.035" rpy=" 0.0  -1.57 0.0"/>
+            <xacro:omni_wheel parent="base_link" child="back_left"   xyz="-0.205  0.255 0.035" rpy="-1.57  0    0.0"/>
+            <xacro:omni_wheel parent="base_link" child="front_right" xyz=" 0.205 -0.255 0.035" rpy=" 1.57  0    0.0"/>
+        </xacro:if>
+        <xacro:unless value="$(arg use_omni_wheel)">
+            <!--Normal Wheels-->
+            <xacro:include filename="wheel.xacro"/>
+            <xacro:wheel parent="base_link" child="front_left"  xyz=" 0.245  0.205 0.035" rpy=" 0.0   1.57 0.0 "/>
+            <xacro:wheel parent="base_link" child="back_right"  xyz="-0.245 -0.205 0.035" rpy=" 0.0  -1.57 0.0"/>
+            <xacro:wheel parent="base_link" child="back_left"   xyz="-0.205  0.245 0.035" rpy="-1.57  0    0.0"/>
+            <xacro:wheel parent="base_link" child="front_right" xyz=" 0.205 -0.245 0.035" rpy=" 1.57  0    0.0"/>
+        </xacro:unless>
     </xacro:if>
-    <xacro:unless value="$(arg use_omni_wheel)">
-        <!--Normal Wheels-->
-        <xacro:include filename="wheel.xacro"/>
-        <xacro:wheel parent="base_link" child="front_left"  xyz=" 0.245   0.205 0.035"  rpy=" 0.0   1.57 0.0 "/>
-        <xacro:wheel parent="base_link" child="back_right"   xyz="-0.245  -0.205 0.035"  rpy=" 0.0  -1.57 0.0"/>
-        <xacro:wheel parent="base_link" child="back_left"   xyz="-0.205  0.245 0.035"   rpy="-1.57  0    0.0"/>
-        <xacro:wheel parent="base_link" child="front_right"  xyz=" 0.205 -0.245 0.035"   rpy=" 1.57  0    0.0"/>
-    </xacro:unless>
+    <!-- Bot ARM -->
+    <xacro:if value="$(arg use_eva)">
+        <xacro:include filename="leg.xacro"/>
+        <xacro:include filename="body.xacro"/>
+        <xacro:include filename="realsense.xacro"/>
+        <xacro:include filename="arm.xacro"/>
+        <xacro:sholder parent="body" child="left"  v_rpy="0.0 0.0 0"    c_xyz="0.0  0.035 0.0" o_xyz="0    0.118 0.457" o_rpy="0.0  0.0  0.0"/>
+        <xacro:sholder parent="body" child="right" v_rpy="0.0 0.0 3.14" c_xyz="0.0 -0.035 0.0" o_xyz="0.0 -0.118 0.457" o_rpy="3.14 3.14 3.14"/>
+        <xacro:upper_biceps side="left"  lower="0"     upper="2.09" o_xyz="0  0.040 0"/>
+        <xacro:upper_biceps side="right" lower="-2.09" upper="0"    o_xyz="0 -0.040 0"/>
+        <xacro:lower_biceps side="left"  lower="-1.57" upper="0"/>
+        <xacro:lower_biceps side="right" lower="0"     upper="1.57"/>
+        <xacro:elbow side="left"  lower="0" upper="-2.05"/>
+        <xacro:elbow side="right" lower="0" upper="-2.05"/>
+        <xacro:wrist side="left"  lower="-1.57" upper="1.57"/>
+        <xacro:wrist side="right" lower="-1.57" upper="1.57"/>
+        <xacro:hand side="left"  lower="-1.10" upper="0.6"/>
+        <xacro:hand side="right" lower="-0.6"  upper="1.10"/>
+    </xacro:if>
 </robot>

Commit message: Update arm.xacro

File: description/arm.xacro (robot description, xacro)
@@ -147,10 +147,10 @@
         </joint>
     </xacro:macro>
-    <xacro:macro name="hand" params="side lower upper">
+    <xacro:macro name="hand" params="side lower upper xyz">
         <link name="${side}_hand">
             <visual>
-                <origin xyz="0.0 0.0 0.0" rpy="0 0 1.57"/>
-                <geometry>
-                    <mesh filename="file://$(find project_eva)/meshes/EVA/Arm/hand.STL"/>
+                <origin xyz="${xyz}" rpy="1.57 3.14 0"/>
+                <geometry>
+                    <mesh filename="file://$(find project_eva)/meshes/EVA/Arm/hand/${side}_palm.STL" scale="0.001 0.001 0.001"/>
                 </geometry>
                 <material name="skin">
@@ -176,3 +176,80 @@
         </joint>
     </xacro:macro>
+<!--/////////////////////////////////////////// FINGERS  /////////////////////////////////////////////////////////////////-->
+    <xacro:macro name="finger_joints" params="name parent child mimic xyz lower upper">
+         <joint name="${name}_joint" type="revolute">
+            <axis xyz="1 0 0"/>
+            <limit effort="0.1" lower="${lower}" upper="${upper}" velocity="0.2"/>
+            <origin xyz="${xyz}" rpy="0 0 0" />
+            <parent link="${parent}" />
+            <child link="${child}" />
+            <mimic joint="${mimic}" multiplier="1"/>
+        </joint>
+    </xacro:macro>
+     <xacro:macro name="finger_joints_1" params="name parent child xyz lower upper">
+         <joint name="${name}_joint" type="revolute">
+            <axis xyz="1 0 0"/>
+            <limit effort="0.1" lower="${lower}" upper="${upper}" velocity="0.2"/>
+            <origin xyz="${xyz}" rpy="0 0 0" />
+            <parent link="${parent}" />
+            <child link="${child}" />
+        </joint>
+    </xacro:macro>
+    <xacro:macro name="finger_link" params="side finger link xyz rpy mesh">
+        <link name="${side}_finger_${finger}_link_${link}">
+            <visual>
+                <origin xyz="${xyz}" rpy="${rpy}"/>
+                <geometry>
+                    <mesh filename="file://$(find project_eva)/meshes/EVA/Arm/Hand/${mesh}.STL" scale="0.001 0.001 0.001"/>
+                </geometry>
+                <material name="skin">
+                    <color rgba="${255/255} ${219/255} ${184/255} 1.0"/>
+                </material>
+            </visual>
+        </link>
+    </xacro:macro>
+    <joint name="right_finger_5_joint_1" type="revolute">
+        <axis xyz="0 0 1"/>
+        <limit effort="0.1"  lower="0" upper="1.57" velocity="0.2"/>
+        <origin xyz="0.044 0.0095 -0.02" rpy="0 0 0" />
+        <parent link="right_hand"/>
+        <child link="right_finger_5_link_1" />
+    </joint>
+    <joint name="right_finger_5_joint_2" type="revolute">
+        <axis xyz="0 1 0"/>
+        <limit effort="0.1"  lower="0" upper="1.22" velocity="0.2"/>
+        <origin xyz="0.02 0.0005 -0.0175" rpy="0 0 0" />
+        <parent link="right_finger_5_link_1" />
+        <child link="right_finger_5_link_2" />
+    </joint>
+    <joint name="right_finger_5_joint_3" type="revolute">
+        <axis xyz="0 1 0"/>
+        <limit effort="0.1"  lower="0" upper="1.22" velocity="0.2"/>
+        <origin xyz="0.019 0 0" rpy="0 0 0" />
+        <parent link="right_finger_5_link_2" />
+        <child link="right_finger_5_link_3" />
+        <mimic joint="right_finger_5_joint_2" multiplier="1"/>
+    </joint>
+    <joint name="left_finger_5_joint_1" type="revolute">
+        <axis xyz="0 0 1"/>
+        <limit effort="0.1"  lower="-1.57" upper="0" velocity="0.2"/>
+        <origin xyz="0.044 -0.0095 -0.02" rpy="0 0 0" />
+        <parent link="left_hand"/>
+        <child link="left_finger_5_link_1" />
+    </joint>
+    <joint name="left_finger_5_joint_2" type="revolute">
+        <axis xyz="0 1 0"/>
+        <limit effort="0.1"  lower="0" upper="1.22" velocity="0.2"/>
+        <origin xyz="0.02 0.0005 -0.0175" rpy="0 0 0" />
+        <parent link="left_finger_5_link_1" />
+        <child link="left_finger_5_link_2" />
+    </joint>
+    <joint name="left_finger_5_joint_3" type="revolute">
+        <axis xyz="0 1 0"/>
+        <limit effort="0.1"  lower="0" upper="1.22" velocity="0.2"/>
+        <origin xyz="0.019 0 0" rpy="0 0 0" />
+        <parent link="left_finger_5_link_2" />
+        <child link="left_finger_5_link_3" />
+        <mimic joint="left_finger_5_joint_2" multiplier="1"/>
+    </joint>
 </robot>

Commit message: Update arm.xacro

File: description/arm.xacro (robot description, xacro)
@@ -152,5 +152,5 @@
                 <origin xyz="${xyz}" rpy="1.57 3.14 0"/>
                 <geometry>
-                    <mesh filename="file://$(find project_eva)/meshes/EVA/Arm/hand/${side}_palm.STL" scale="0.001 0.001 0.001"/>
+                    <mesh filename="file://$(find project_eva)/meshes/EVA/Arm/Hand/${side}_palm.STL" scale="0.001 0.001 0.001"/>
                 </geometry>
                 <material name="skin">
